Commit message: Wait for random target

File: src/fun4/robot/visual/my-robot.xacro (robot description, xacro)
@@ -4,5 +4,5 @@
     <visual>
       <geometry>
-        <mesh filename="file:///$(find example_description)/meshes/link_0.stl"/>
+        <mesh filename="file:///$(find fun4)/meshes/link_0.stl"/>
       </geometry>
     </visual>
@@ -11,5 +11,5 @@
     <visual>
       <geometry>
-        <mesh filename="file:///$(find example_description)/meshes/link_1.stl"/>
+        <mesh filename="file:///$(find fun4)/meshes/link_1.stl"/>
       </geometry>
     </visual>
@@ -30,5 +30,5 @@
       <origin xyz="0.0 0.0 0.0" rpy="0 0 0"/>
       <geometry>
-        <mesh filename="file:///$(find example_description)/meshes/link_2.stl"/>
+        <mesh filename="file:///$(find fun4)/meshes/link_2.stl"/>
       </geometry>
     </visual>
@@ -49,5 +49,5 @@
       <origin xyz="0.0 0.0 0.0" rpy="0 0 0"/>
       <geometry>
-        <mesh filename="file:///$(find example_description)/meshes/link_3.stl"/>
+        <mesh filename="file:///$(find fun4)/meshes/link_3.stl"/>
       </geometry>
     </visual>
@@ -68,5 +68,5 @@
       <origin xyz="0.0 0.0 0.0" rpy="0 0 0"/>
       <geometry>
-        <mesh filename="file:///$(find example_description)/meshes/end_effector.stl"/>
+        <mesh filename="file:///$(find fun4)/meshes/end_effector.stl"/>
       </geometry>
     </visual>
